Commit message: test succeed, but dbc may be false

File: data_fusion/urdf/fusion.urdf (robot description, URDF)
Before this commit: robot test_car, 12 links, 11 joints
Joints:
- joint lidar_velo: origin xyz=1.88 0 2.166  rpy=0 0 0 -> xyz=0.88 0 2.166  rpy=0 0 -1.57075

Commit message: changed sth

File: data_fusion/urdf/fusion.urdf (robot description, URDF)
Before this commit: robot test_car, 12 links, 11 joints
Joints:
- joint lidar_ibeo: type continuous -> fixed
- joint lidar_velo: type continuous -> fixed
- joint radar: type continuous -> fixed
- joint radar_0: type continuous -> fixed
- joint radar_1: type continuous -> fixed
- joint radar_2: type continuous -> fixed
- joint radar_3: type continuous -> fixed

Commit message: ibeo_had refined

File: data_fusion/urdf/fusion.urdf (robot description, URDF)
Before this commit: robot test_car, 12 links, 11 joints
Joints:
- joint radar: origin xyz=3.617 -0.009 0.431  rpy=0 0 0 -> xyz=3.95 0 0.431  rpy=0 0 -1.57075
- joint radar_0: origin xyz=3.514 0.669 0.16  rpy=0 0 -0.6108 -> xyz=3.514 0.669 0.16  rpy=0 0 0.6108
- joint radar_1: origin xyz=3.515 -0.669 0.16  rpy=0 0 0.6108 -> xyz=3.515 -0.669 0.16  rpy=0 0 -0.6108
